File: TxBoard.kicad_pcb (KiCad board)
At the start: 2 copper layers, 94 x 31.8 mm, 22 parts, among them J1 RCA Socket, Q1 RU1J002YNTCL, SW1 Pull-Up, SW2 Input(Hi-Z)/Output, SW3 Low/High

Commit message: Cost reduction
dont wanna pay for no order number, so just put it where it is not visible
Other:
- board text added: "JLCJLCJLCJLC"
Changed lines of the file:
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@@
   (gr_line (start 126.492 94.615) (end 126.492 97.155) (layer "F.SilkS") (width 0.16))
   (gr_rect (start 102.997 81.28) (end 196.977 113.03) (layer "Edge.Cuts") (width 0.1) (fill none))
+  (gr_text "JLCJLCJLCJLC" (at 141.72 91.7) (layer "B.SilkS")
+    (effects (font (size 1.5 1.5) (thickness 0.16)) (justify mirror))
+  )
   (gr_text "Revision 1\n4/19/22" (at 108.1 96.725) (layer "B.SilkS")
     (effects (font (size 1 1) (thickness 0.16)) (justify mirror))

Commit message: Lessons learned
>:(
Parts:
- removed BZ1: Buzzer, PKM13EPYH4000-A0:SPKR_PKM13EPYH4000-A0
- removed R4: 150Ω, Resistor_SMD:R_0603_1608Metric_Pad0.98x0.95mm_HandSolder
- added D2: Red, LED_SMD:LED_0603_1608Metric_Pad1.05x0.95mm_HandSolder, F.Cu at (178.1, 90.6)
- D1: value LED -> Green
- SW1, SW2: footprint EG1218:EG1218 -> JS102011SCQN:JS102011SCQN
- SW3: value Low/High -> High/Low; footprint EG1218:EG1218 -> JS102011SCQN:JS102011SCQN
- moved SW2 2.55 mm to (146.8, 97.2), turned to 0 degrees
- moved C1 2.48 mm to (183.7, 96.3)
- moved SW3 2.45 mm to (127.8, 97.2), turned to 0 degrees
- moved SW1 2.02 mm to (165.8, 97.2), turned to 0 degrees
- moved J1 1.84 mm to (192.6, 97.2)
- moved G*** 1.71 mm to (156.4, 84.8)
- moved REF** 0.59 mm to (108.1, 97.2)
Connections:
- REF** pad 1: (no net) -> GND (x4)
Routing:
- net Net-(R3-Pad2): track 44.8 -> 50.1 mm, vias 0 -> 1
- net Net-(R2-Pad2): track 8.16 -> 13.1 mm, vias 0 -> 1
- net +BATT: track 159.6 -> 155.7 mm, vias 1 -> 2
- net Net-(C1-Pad1): track 52.5 -> 49.9 mm
- net Net-(SW3-Pad1): track 85.2 -> 83.4 mm, vias 2 -> 4
Other:
- board text added: "High"
- board text added: "Short"
- board text removed: "High 150Ω"

Commit message: Design review 2
good 4 prototype 2
Parts:
- moved TP1 23.5 mm to (173.5, 85.4)
- moved TP2 19.4 mm to (173.6, 88.5)
- moved REF** 2.70 mm to (189.2, 86.4)
- moved REF** 2.60 mm to (189.3, 108.0)
Routing:
- net +BATT: track 155.7 -> 90.6 mm
- net Net-(SW3-Pad1): track 83.4 -> 68.5 mm, vias 4 -> 2
Other:
- board size 94 x 31.8 mm -> 94 x 31.7 mm
- board text added: "Revision 2 5/7/22"
- board text removed: "Permanent Marker"
- board text removed: "Revision 1 4/19/22"

Commit message: where was I
oh yeah
Parts:
- added C2: 10μF, Capacitor_SMD:C_0805_2012Metric_Pad1.18x1.45mm_HandSolder, B.Cu at (183.7, 90.6)
Routing:
- net Net-(C2-Pad2): track 68.5 -> 70.8 mm
Other:
- board text added: "Revision 3 5/28/22"
- board text removed: "Revision 2 5/7/22"
Changed lines of the file:
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@@
   (title_block
     (title "TixBoard Communications Education Board")
-    (date "2022-04-16")
-    (rev "3")
+    (date "2022-05-28")
+    (rev "4")
     (company "QuarterWave Engineering")
   )
@@
     (pad_to_mask_clearance 0)
     (pcbplotparams
-      (layerselection 0x00010f0_ffffffff)
+      (layerselection 0x00010fc_ffffffff)
       (disableapertmacros false)
       (usegerberextensions true)
@@
       (svgprecision 6)
       (excludeedgelayer false)
-      (plotframeref true)
+      (plotframeref false)
       (viasonmask false)
       (mode 1)
@@
       (psa4output false)
       (plotreference true)
-      (plotvalue true)
+      (plotvalue false)
       (plotinvisibletext false)
       (sketchpadsonfab false)
       (subtractmaskfromsilk true)
-      (outputformat 4)
+      (outputformat 1)
       (mirror false)
       (drillshape 0)
@@
   (net 6 "Net-(R2-Pad2)")
   (net 7 "Net-(R3-Pad2)")
-  (net 8 "Net-(SW3-Pad1)")
+  (net 8 "Net-(C2-Pad2)")
   (net 9 "unconnected-(SW1-Pad3)")
   (net 10 "Net-(SW2-Pad1)")
@@
     (fp_line (start -0.5 -0.4) (end -0.8 -0.1) (layer "F.Fab") (width 0.1))
     (pad "1" smd roundrect (at -0.875 0 180) (size 1.05 0.95) (layers "F.Cu" "F.Paste" "F.Mask") (roundrect_rratio 0.25)
-      (net 8 "Net-(SW3-Pad1)") (pinfunction "K") (pintype "passive"))
+      (net 8 "Net-(C2-Pad2)") (pinfunction "K") (pintype "passive"))
     (pad "2" smd roundrect (at 0.875 0 180) (size 1.05 0.95) (layers "F.Cu" "F.Paste" "F.Mask") (roundrect_rratio 0.25)
       (net 4 "+BATT") (pinfunction "A") (pintype "passive"))
@@
     (fp_arc (start 0.3048 -4.2545) (mid 0 -3.9497) (end -0.3048 -4.2545) (layer "F.Fab") (width 0.1))
     (pad "1" smd rect (at -2.85 -2.5) (size 2.7 1) (layers "F.Cu" "F.Paste" "F.Mask")
-      (net 8 "Net-(SW3-Pad1)") (pinfunction "A") (pintype "passive"))
+      (net 8 "Net-(C2-Pad2)") (pinfunction "A") (pintype "passive"))
     (pad "2" smd rect (at 2.85 0) (size 2.7 1) (layers "F.Cu" "F.Paste" "F.Mask")
       (net 10 "Net-(SW2-Pad1)") (pinfunction "B") (pintype "passive"))
@@
       (net 2 "GND"))
   )
+  (footprint "Capacitor_SMD:C_0805_2012Metric_Pad1.18x1.45mm_HandSolder" (layer "B.Cu")
+    (at 183.7 90.6 180)
+    (descr "Capacitor SMD 0805 (2012 Metric), square (rectangular) end terminal, IPC_7351 nominal with elongated pad for handsoldering. (Body size source: IPC-SM-782 page 76, https://www.pcb-3d.com/wordpress/wp-content/uploads/ipc-sm-782a_amendment_1_and_2.pdf, https://docs.google.com/spreadsheets/d/1BsfQQcO9C6DZCsRaXUlFlo91Tg2WpOkGARC1WS5S8t0/edit?usp=sharing), generated with kicad-footprint-generator")
+    (tags "capacitor handsolder")
+    (property "Sheetfile" "TxBoard.kicad_sch")
+    (property "Sheetname" "")
+    (attr smd)
+    (fp_text reference "C2" (at 0 1.7) (layer "B.SilkS")
+      (effects (font (size 1 1) (thickness 0.15)) (justify mirror))
+    )
+    (fp_text value "10μF" (at 0 -1.68) (layer "B.Fab")
+      (effects (font (size 1 1) (thickness 0.15)) (justify mirror))
+    )
+    (fp_text user "${REFERENCE}" (at 0 0) (layer "B.Fab")
+      (effects (font (size 0.5 0.5) (thickness 0.08)) (justify mirror))
+    )
+    (fp_line (start -0.261252 -0.735) (end 0.261252 -0.735) (layer "B.SilkS") (width 0.12))
+    (fp_line (start -0.261252 0.735) (end 0.261252 0.735) (layer "B.SilkS") (width 0.12))
+    (fp_line (start -1.88 0.98) (end 1.88 0.98) (layer "B.CrtYd") (width 0.05))
+    (fp_line (start 1.88 0.98) (end 1.88 -0.98) (layer "B.CrtYd") (width 0.05))
+    (fp_line (start -1.88 -0.98) (end -1.88 0.98) (layer "B.CrtYd") (width 0.05))
+    (fp_line (start 1.88 -0.98) (end -1.88 -0.98) (layer "B.CrtYd") (width 0.05))
+    (fp_line (start 1 0.625) (end 1 -0.625) (layer "B.Fab") (width 0.1))
+    (fp_line (start -1 -0.625) (end -1 0.625) (layer "B.Fab") (width 0.1))
+    (fp_line (start 1 -0.625) (end -1 -0.625) (layer "B.Fab") (width 0.1))
+    (fp_line (start -1 0.625) (end 1 0.625) (layer "B.Fab") (width 0.1))
+    (pad "1" smd roundrect (at -1.0375 0 180) (size 1.175 1.45) (layers "B.Cu" "B.Paste" "B.Mask") (roundrect_rratio 0.2127659574)
+      (net 2 "GND") (pintype "passive"))
+    (pad "2" smd roundrect (at 1.0375 0 180) (size 1.175 1.45) (layers "B.Cu" "B.Paste" "B.Mask") (roundrect_rratio 0.2127659574)
+      (net 8 "Net-(C2-Pad2)") (pintype "passive"))
+    (model "${KICAD6_3DMODEL_DIR}/Capacitor_SMD.3dshapes/C_0805_2012Metric.wrl"
+      (offset (xyz 0 0 0))
+      (scale (xyz 1 1 1))
+      (rotate (xyz 0 0 0))
+    )
+  )
   (footprint "KLPX-0848A-2-B:KLPX-0848A-2-B" (layer "B.Cu")
     (at 192.6 97.155 90)
@@
     (effects (font (size 1.5 1.5) (thickness 0.16)) (justify mirror))
   )
-  (gr_text "Revision 2\n5/7/22" (at 108.1 96.725) (layer "B.SilkS")
+  (gr_text "Revision 3\n5/28/22" (at 108.1 96.725) (layer "B.SilkS")
     (effects (font (size 1 1) (thickness 0.16)) (justify mirror))
   )
@@
   (segment (start 176.65 94.35) (end 176.65 101.25) (width 0.381) (layer "B.Cu") (net 8))
   (segment (start 176.1 101.8) (end 135 101.8) (width 0.381) (layer "B.Cu") (net 8))
+  (segment (start 182.6625 90.6) (end 180.4 90.6) (width 0.381) (layer "B.Cu") (net 8))
   (segment (start 176.65 101.25) (end 176.1 101.8) (width 0.381) (layer "B.Cu") (net 8))
   (segment (start 180.4 90.6) (end 176.65 94.35) (width 0.381) (layer "B.Cu") (net 8))
