File: TxBoard.kicad_sch (KiCad schematic)
At the start: 15 parts, among them J1 RCA Socket, Q1 RU1J002YNTCL, SW1 Pull-Up, SW2 Input(Hi-Z)/Output, SW3 Low/High

Commit message: Lessons learned
>:(
Parts:
- removed BZ1: Buzzer, PKM13EPYH4000-A0:SPKR_PKM13EPYH4000-A0, symbol Device:Buzzer
- removed R4: 150Ω, Resistor_SMD:R_0603_1608Metric_Pad0.98x0.95mm_HandSolder, symbol Device:R_Small_US
- added D2: Red, LED_SMD:LED_0603_1608Metric_Pad1.05x0.95mm_HandSolder, symbol Device:LED
- D1: value LED -> Green
- SW1, SW2: footprint EG1218:EG1218 -> JS102011SCQN:JS102011SCQN
- SW3: value Low/High -> High/Low; footprint EG1218:EG1218 -> JS102011SCQN:JS102011SCQN
Connections:
- net +BATT: now also D2.2 (A)
- net at SW3.1 (A): now also D2.1 (K)
Changed lines of the file:
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@@
     (title "TixBoard Communications Education Board")
     (date "2022-04-14")
-    (rev "2")
+    (rev "3")
     (company "QuarterWave Engineering")
     (comment 2 "Design Changes: Cost reduction, MOSFET changed to more suitable model with lower Vth")
@@
     (comment 4 "[Designed with <3 in San Diego - Licensed under MIT License]")
   )
-  (junction (at 120.65 87.63) (diameter 0) (color 0 0 0 0)
-  )
   (junction (at 154.94 104.14) (diameter 0) (color 0 0 0 0)
-  )
-  (junction (at 120.65 82.55) (diameter 0) (color 0 0 0 0)
   )
   (junction (at 173.99 104.14) (diameter 0) (color 0 0 0 0)
@@
     (stroke (width 0) (type default) (color 0 0 0 0))
   )
-  (wire (pts (xy 116.84 82.55) (xy 120.65 82.55))
-    (stroke (width 0) (type default) (color 0 0 0 0))
-  )
   (wire (pts (xy 149.86 109.22) (xy 149.86 113.03))
     (stroke (width 0) (type default) (color 0 0 0 0))
   )
+  (wire (pts (xy 120.65 92.71) (xy 129.54 92.71))
+    (stroke (width 0) (type default) (color 0 0 0 0))
+  )
   (wire (pts (xy 139.7 95.25) (xy 144.78 95.25))
     (stroke (width 0) (type default) (color 0 0 0 0))
   )
+  (wire (pts (xy 120.65 78.74) (xy 120.65 81.28))
+    (stroke (width 0) (type default) (color 0 0 0 0))
+  )
   (wire (pts (xy 185.42 95.25) (xy 185.42 99.06))
     (stroke (width 0) (type default) (color 0 0 0 0))
@@
     (stroke (width 0) (type default) (color 0 0 0 0))
   )
-  (wire (pts (xy 120.65 87.63) (xy 120.65 92.71))
-    (stroke (width 0) (type default) (color 0 0 0 0))
-  )
   (wire (pts (xy 173.99 104.14) (xy 177.8 104.14))
     (stroke (width 0) (type default) (color 0 0 0 0))
@@
     (stroke (width 0) (type default) (color 0 0 0 0))
   )
-  (wire (pts (xy 120.65 78.74) (xy 120.65 82.55))
-    (stroke (width 0) (type default) (color 0 0 0 0))
-  )
   (wire (pts (xy 185.42 109.22) (xy 185.42 113.03))
     (stroke (width 0) (type default) (color 0 0 0 0))
   )
-  (wire (pts (xy 129.54 92.71) (xy 120.65 92.71))
-    (stroke (width 0) (type default) (color 0 0 0 0))
-  )
-  (wire (pts (xy 116.84 87.63) (xy 120.65 87.63))
-    (stroke (width 0) (type default) (color 0 0 0 0))
-  )
   (wire (pts (xy 166.37 104.14) (xy 166.37 101.6))
     (stroke (width 0) (type default) (color 0 0 0 0))
@@
   )
   (wire (pts (xy 173.99 107.95) (xy 173.99 104.14))
+    (stroke (width 0) (type default) (color 0 0 0 0))
+  )
+  (wire (pts (xy 120.65 88.9) (xy 120.65 92.71))
     (stroke (width 0) (type default) (color 0 0 0 0))
   )
@@
       (effects (font (size 1.27 1.27)) (justify right))
     )
-    (property "Value" "LED" (id 1) (at 188.341 85.8397 90)
+    (property "Value" "Green" (id 1) (at 188.341 85.8397 90)
       (effects (font (size 1.27 1.27)) (justify right))
     )
@@
     (in_bom yes) (on_board yes) (fields_autoplaced)
     (property "Reference" "SW3" (id 0) (at 134.62 88.6292 0))
-    (property "Value" "Low/High" (id 1) (at 134.62 91.1661 0))
-    (property "Footprint" "EG1218:EG1218" (id 2) (at 134.62 95.25 0)
+    (property "Value" "High/Low" (id 1) (at 134.62 91.1661 0))
+    (property "Footprint" "JS102011SCQN:JS102011SCQN" (id 2) (at 134.62 95.25 0)
       (effects (font (size 1.27 1.27)) hide)
     )
@@
       (effects (font (size 1.27 1.27)) (justify right))
     )
-    (property "Footprint" "EG1218:EG1218" (id 2) (at 166.37 96.52 0)
+    (property "Footprint" "JS102011SCQN:JS102011SCQN" (id 2) (at 166.37 96.52 0)
       (effects (font (size 1.27 1.27)) hide)
     )
@@
     )
     (pin "1")
-  )
-  (symbol (lib_id "Device:Buzzer") (at 114.3 85.09 0) (mirror y) (unit 1)
-    (in_bom yes) (on_board yes)
-    (property "Reference" "BZ1" (id 0) (at 114.3 78.74 0))
-    (property "Value" "Buzzer" (id 1) (at 114.3 90.17 0))
-    (property "Footprint" "PKM13EPYH4000-A0:SPKR_PKM13EPYH4000-A0" (id 2) (at 114.935 82.55 90)
-      (effects (font (size 1.27 1.27)) hide)
-    )
-    (property "Datasheet" "~" (id 3) (at 114.935 82.55 90)
-      (effects (font (size 1.27 1.27)) hide)
-    )
-    (pin "1")
-    (pin "2")
   )
   (symbol (lib_id "Device:R_Small_US") (at 163.83 83.82 0) (unit 1)
@@
     (property "Reference" "SW2" (id 0) (at 149.86 91.1692 0))
     (property "Value" "Input(Hi-Z)/Output" (id 1) (at 149.86 93.7061 0))
-    (property "Footprint" "EG1218:EG1218" (id 2) (at 149.86 97.79 0)
+    (property "Footprint" "JS102011SCQN:JS102011SCQN" (id 2) (at 149.86 97.79 0)
       (effects (font (size 1.27 1.27)) hide)
     )
@@
     )
     (pin "1")
+  )
+  (symbol (lib_id "Device:LED") (at 120.65 85.09 90) (unit 1)
+    (in_bom yes) (on_board yes)
+    (property "Reference" "D2" (id 0) (at 114.3 85.09 90)
+      (effects (font (size 1.27 1.27)) (justify right))
+    )
+    (property "Value" "Red" (id 1) (at 114.3 87.63 90)
+      (effects (font (size 1.27 1.27)) (justify right))
+    )
+    (property "Footprint" "LED_SMD:LED_0603_1608Metric_Pad1.05x0.95mm_HandSolder" (id 2) (at 120.65 85.09 0)
+      (effects (font (size 1.27 1.27)) hide)
+    )
+    (property "Datasheet" "~" (id 3) (at 120.65 85.09 0)
+      (effects (font (size 1.27 1.27)) hide)
+    )
+    (pin "1")
+    (pin "2")
   )
   (symbol (lib_id "power:GND") (at 120.65 113.03 0) (unit 1)
@@
     )
     (pin "1")
-  )
-  (symbol (lib_id "Device:R_Small_US") (at 120.65 85.09 0) (unit 1)
-    (in_bom yes) (on_board yes) (fields_autoplaced)
-    (property "Reference" "R4" (id 0) (at 122.301 84.2553 0)
-      (effects (font (size 1.27 1.27)) (justify left))
-    )
-    (property "Value" "150Ω" (id 1) (at 122.301 86.7922 0)
-      (effects (font (size 1.27 1.27)) (justify left))
-    )
-    (property "Footprint" "Resistor_SMD:R_0603_1608Metric_Pad0.98x0.95mm_HandSolder" (id 2) (at 120.65 85.09 0)
-      (effects (font (size 1.27 1.27)) hide)
-    )
-    (property "Datasheet" "~" (id 3) (at 120.65 85.09 0)
-      (effects (font (size 1.27 1.27)) hide)
-    )
-    (pin "1")
-    (pin "2")
   )
   (sheet_instances
@@
       (reference "BT1") (unit 1) (value "2xAA") (footprint "BC2AAPC:BAT_BC2AAPC")
     )
-    (path "/cee8c350-8be0-477d-80d4-b88d2f05177c"
-      (reference "BZ1") (unit 1) (value "Buzzer") (footprint "PKM13EPYH4000-A0:SPKR_PKM13EPYH4000-A0")
-    )
     (path "/6942edd1-0ba6-453d-957e-b3b7fa528bf9"
       (reference "C1") (unit 1) (value "10μF") (footprint "Capacitor_SMD:C_0805_2012Metric_Pad1.18x1.45mm_HandSolder")
     )
     (path "/1cd534f3-3a3a-4350-959a-ea3b2fc71750"
-      (reference "D1") (unit 1) (value "LED") (footprint "LED_SMD:LED_0603_1608Metric_Pad1.05x0.95mm_HandSolder")
+      (reference "D1") (unit 1) (value "Green") (footprint "LED_SMD:LED_0603_1608Metric_Pad1.05x0.95mm_HandSolder")
+    )
+    (path "/e117b9a3-4868-45c7-860c-7a0459b0683b"
+      (reference "D2") (unit 1) (value "Red") (footprint "LED_SMD:LED_0603_1608Metric_Pad1.05x0.95mm_HandSolder")
     )
     (path "/1ba46d81-748c-4295-a4f1-72252a533537"
@@
       (reference "R3") (unit 1) (value "150Ω") (footprint "Resistor_SMD:R_0603_1608Metric_Pad0.98x0.95mm_HandSolder")
     )
-    (path "/fa7dc726-d91e-4f17-a069-0c12165ed6d6"
-      (reference "R4") (unit 1) (value "150Ω") (footprint "Resistor_SMD:R_0603_1608Metric_Pad0.98x0.95mm_HandSolder")
-    )
     (path "/c573f4f3-c4fc-4aca-ad6c-946df532b32a"
-      (reference "SW1") (unit 1) (value "Pull-Up") (footprint "EG1218:EG1218")
+      (reference "SW1") (unit 1) (value "Pull-Up") (footprint "JS102011SCQN:JS102011SCQN")
     )
     (path "/d2aeeca3-2d6b-49ff-8e68-e891d2132e85"
-      (reference "SW2") (unit 1) (value "Input(Hi-Z)/Output") (footprint "EG1218:EG1218")
+      (reference "SW2") (unit 1) (value "Input(Hi-Z)/Output") (footprint "JS102011SCQN:JS102011SCQN")
     )
     (path "/c3265d8f-1789-4158-aa57-27936cdaa040"
-      (reference "SW3") (unit 1) (value "Low/High") (footprint "EG1218:EG1218")
+      (reference "SW3") (unit 1) (value "High/Low") (footprint "JS102011SCQN:JS102011SCQN")
     )
     (path "/cd78a05f-3030-4df8-a06c-277f5becd950"

Commit message: where was I
oh yeah
Parts:
- added C2: 10μF, Capacitor_SMD:C_0805_2012Metric_Pad1.18x1.45mm_HandSolder, symbol Device:C_Small
Connections:
- net GND: now also C2.1
- net at D2.1 (K), SW3.1 (A): now also C2.2
Changed lines of the file:
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@@
   (title_block
     (title "TixBoard Communications Education Board")
-    (date "2022-04-14")
-    (rev "3")
+    (date "2022-05-28")
+    (rev "4")
     (company "QuarterWave Engineering")
     (comment 2 "Design Changes: Cost reduction, MOSFET changed to more suitable model with lower Vth")
@@
   (junction (at 166.37 104.14) (diameter 0) (color 0 0 0 0)
   )
+  (junction (at 120.65 92.71) (diameter 0) (color 0 0 0 0)
+  )
   (no_connect (at 144.78 100.33))
   (no_connect (at 168.91 91.44))
@@
     (stroke (width 0) (type default) (color 0 0 0 0))
   )
+  (wire (pts (xy 120.65 92.71) (xy 129.54 92.71))
+    (stroke (width 0) (type default) (color 0 0 0 0))
+  )
   (wire (pts (xy 149.86 109.22) (xy 149.86 113.03))
     (stroke (width 0) (type default) (color 0 0 0 0))
   )
-  (wire (pts (xy 120.65 92.71) (xy 129.54 92.71))
+  (wire (pts (xy 119.38 92.71) (xy 120.65 92.71))
+    (stroke (width 0) (type default) (color 0 0 0 0))
+  )
+  (wire (pts (xy 120.65 88.9) (xy 120.65 92.71))
     (stroke (width 0) (type default) (color 0 0 0 0))
   )
@@
     (stroke (width 0) (type default) (color 0 0 0 0))
   )
+  (wire (pts (xy 114.3 92.71) (xy 111.76 92.71))
+    (stroke (width 0) (type default) (color 0 0 0 0))
+  )
+  (wire (pts (xy 111.76 92.71) (xy 111.76 113.03))
+    (stroke (width 0) (type default) (color 0 0 0 0))
+  )
   (wire (pts (xy 120.65 105.41) (xy 120.65 113.03))
     (stroke (width 0) (type default) (color 0 0 0 0))
@@
   )
   (wire (pts (xy 173.99 107.95) (xy 173.99 104.14))
-    (stroke (width 0) (type default) (color 0 0 0 0))
-  )
-  (wire (pts (xy 120.65 88.9) (xy 120.65 92.71))
     (stroke (width 0) (type default) (color 0 0 0 0))
   )
@@
     (pin "2")
   )
+  (symbol (lib_id "power:GND") (at 111.76 113.03 0) (unit 1)
+    (in_bom yes) (on_board yes) (fields_autoplaced)
+    (property "Reference" "#PWR0112" (id 0) (at 111.76 119.38 0)
+      (effects (font (size 1.27 1.27)) hide)
+    )
+    (property "Value" "GND" (id 1) (at 111.76 117.4734 0))
+    (property "Footprint" "" (id 2) (at 111.76 113.03 0)
+      (effects (font (size 1.27 1.27)) hide)
+    )
+    (property "Datasheet" "" (id 3) (at 111.76 113.03 0)
+      (effects (font (size 1.27 1.27)) hide)
+    )
+    (pin "1")
+  )
   (symbol (lib_id "Switch:SW_SPDT") (at 149.86 97.79 0) (mirror y) (unit 1)
     (in_bom yes) (on_board yes) (fields_autoplaced)
@@
   (symbol (lib_id "Device:LED") (at 120.65 85.09 90) (unit 1)
     (in_bom yes) (on_board yes)
-    (property "Reference" "D2" (id 0) (at 114.3 85.09 90)
-      (effects (font (size 1.27 1.27)) (justify right))
-    )
-    (property "Value" "Red" (id 1) (at 114.3 87.63 90)
+    (property "Reference" "D2" (id 0) (at 115.57 83.82 90)
+      (effects (font (size 1.27 1.27)) (justify right))
+    )
+    (property "Value" "Red" (id 1) (at 115.57 86.36 90)
       (effects (font (size 1.27 1.27)) (justify right))
     )
@@
     )
     (property "Datasheet" "~" (id 3) (at 120.65 85.09 0)
+      (effects (font (size 1.27 1.27)) hide)
+    )
+    (pin "1")
+    (pin "2")
+  )
+  (symbol (lib_id "Device:C_Small") (at 116.84 92.71 90) (unit 1)
+    (in_bom yes) (on_board yes)
+    (property "Reference" "C2" (id 0) (at 116.84 90.17 90))
+    (property "Value" "10μF" (id 1) (at 116.84 95.25 90))
+    (property "Footprint" "Capacitor_SMD:C_0805_2012Metric_Pad1.18x1.45mm_HandSolder" (id 2) (at 116.84 92.71 0)
+      (effects (font (size 1.27 1.27)) hide)
+    )
+    (property "Datasheet" "~" (id 3) (at 116.84 92.71 0)
       (effects (font (size 1.27 1.27)) hide)
     )
@@
       (reference "#PWR0111") (unit 1) (value "+BATT") (footprint "")
     )
+    (path "/cfce927e-3248-4d81-8247-6fe1704275b0"
+      (reference "#PWR0112") (unit 1) (value "GND") (footprint "")
+    )
     (path "/4b955b5c-03e5-4624-b491-59cac36331e9"
       (reference "BT1") (unit 1) (value "2xAA") (footprint "BC2AAPC:BAT_BC2AAPC")
@@
       (reference "C1") (unit 1) (value "10μF") (footprint "Capacitor_SMD:C_0805_2012Metric_Pad1.18x1.45mm_HandSolder")
     )
+    (path "/e1a72832-6a60-4b01-92cd-3bc245b7b6d4"
+      (reference "C2") (unit 1) (value "10μF") (footprint "Capacitor_SMD:C_0805_2012Metric_Pad1.18x1.45mm_HandSolder")
+    )
     (path "/1cd534f3-3a3a-4350-959a-ea3b2fc71750"
